Commit message: sim bot with realsense d455

File: src/realsense-ros-gazebo/realsense-ros/realsense2_description/urdf/_d435.urdf.xacro (robot description, xacro)
@@ -9,41 +9,43 @@
   <!-- Includes -->
   <xacro:include filename="$(find realsense2_description)/urdf/_d435.gazebo.xacro" />
-  <xacro:include filename="$(find realsense2_description)/urdf/_materials.urdf.xacro" />
+  <!-- <xacro:include filename="$(find realsense2_description)/urdf/_materials.urdf.xacro" /> -->
   <xacro:include filename="$(find realsense2_description)/urdf/_usb_plug.urdf.xacro" />
-  <xacro:macro name="sensor_d435" params="parent *origin name:=camera use_nominal_extrinsics:=false add_plug:=false use_mesh:=true topics_ns:=camera publish_pointcloud:=true">
+  <xacro:macro name="sensor_d435"
+    params="parent *origin name:=camera use_nominal_extrinsics:=false add_plug:=false use_mesh:=true topics_ns:=camera publish_pointcloud:=true">
     <xacro:property name="M_PI" value="3.1415926535897931" />
     <!-- The following values are approximate, and the camera node
      publishing TF values with actual calibrated camera extrinsic values -->
-    <xacro:property name="d435_cam_depth_to_infra1_offset" value="0.0"/>
-    <xacro:property name="d435_cam_depth_to_infra2_offset" value="-0.050"/>
-    <xacro:property name="d435_cam_depth_to_color_offset" value="0.015"/>
+    <xacro:property name="d435_cam_depth_to_infra1_offset" value="0.0" />
+    <xacro:property name="d435_cam_depth_to_infra2_offset" value="-0.050" />
+    <xacro:property name="d435_cam_depth_to_color_offset" value="0.015" />
     <!-- The following values model the aluminum peripherial case for the
   	D435 camera, with the camera joint represented by the actual
   	peripherial camera tripod mount -->
-    <xacro:property name="d435_cam_width" value="0.090"/>
-    <xacro:property name="d435_cam_height" value="0.025"/>
-    <xacro:property name="d435_cam_depth" value="0.02505"/>
-    <xacro:property name="d435_cam_mount_from_center_offset" value="0.0149"/>
+    <xacro:property name="d435_cam_width" value="0.090" />
+    <xacro:property name="d435_cam_height" value="0.025" />
+    <xacro:property name="d435_cam_depth" value="0.02505" />
+    <xacro:property name="d435_cam_mount_from_center_offset" value="0.0149" />
     <!-- glass cover is 0.1 mm inwards from front aluminium plate -->
-    <xacro:property name="d435_glass_to_front" value="0.1e-3"/>
+    <xacro:property name="d435_glass_to_front" value="0.1e-3" />
     <!-- see datasheet Revision 007, Fig. 4-4 page 65 -->
-    <xacro:property name="d435_zero_depth_to_glass" value="4.2e-3"/>
+    <xacro:property name="d435_zero_depth_to_glass" value="4.2e-3" />
     <!-- convenience precomputation to avoid clutter-->
-    <xacro:property name="d435_mesh_x_offset" value="${d435_cam_mount_from_center_offset-d435_glass_to_front-d435_zero_depth_to_glass}"/>
+    <xacro:property name="d435_mesh_x_offset"
+      value="${d435_cam_mount_from_center_offset-d435_glass_to_front-d435_zero_depth_to_glass}" />
     <!-- The following offset is relative the the physical D435 camera peripherial
   	camera tripod mount -->
-    <xacro:property name="d435_cam_depth_px" value="${d435_cam_mount_from_center_offset}"/>
-    <xacro:property name="d435_cam_depth_py" value="0.0175"/>
-    <xacro:property name="d435_cam_depth_pz" value="${d435_cam_height/2}"/>
+    <xacro:property name="d435_cam_depth_px" value="${d435_cam_mount_from_center_offset}" />
+    <xacro:property name="d435_cam_depth_py" value="0.0175" />
+    <xacro:property name="d435_cam_depth_pz" value="${d435_cam_height/2}" />
     <!-- camera body, with origin at bottom screw mount -->
     <joint name="${name}_joint" type="fixed">
       <xacro:insert_block name="origin" />
-      <parent link="${parent}"/>
+      <parent link="${parent}" />
       <child link="${name}_bottom_screw_frame" />
     </joint>
-    <link name="${name}_bottom_screw_frame"/>
+    <link name="${name}_bottom_screw_frame" />
     <joint name="${name}_link_joint" type="fixed">
-      <origin xyz="${d435_mesh_x_offset} ${d435_cam_depth_py} ${d435_cam_depth_pz}" rpy="0 0 0"/>
-      <parent link="${name}_bottom_screw_frame"/>
+      <origin xyz="${d435_mesh_x_offset} ${d435_cam_depth_py} ${d435_cam_depth_pz}" rpy="0 0 0" />
+      <parent link="${name}_bottom_screw_frame" />
       <child link="${name}_link" />
     </joint>
@@ -52,5 +54,6 @@
         <xacro:if value="${use_mesh}">
           <!-- the mesh origin is at front plate in between the two infrared camera axes -->
-          <origin xyz="${d435_zero_depth_to_glass + d435_glass_to_front} ${-d435_cam_depth_py} 0" rpy="${M_PI/2} 0 ${M_PI/2}"/>
+          <origin xyz="${d435_zero_depth_to_glass + d435_glass_to_front} ${-d435_cam_depth_py} 0"
+            rpy="${M_PI/2} 0 ${M_PI/2}" />
           <geometry>
             <mesh filename="package://realsense2_description/meshes/d435.dae" />
@@ -58,15 +61,15 @@
         </xacro:if>
         <xacro:unless value="${use_mesh}">
-          <origin xyz="0 ${-d435_cam_depth_py} 0" rpy="0 0 0"/>
+          <origin xyz="0 ${-d435_cam_depth_py} 0" rpy="0 0 0" />
           <geometry>
-            <box size="${d435_cam_depth} ${d435_cam_width} ${d435_cam_height}"/>
+            <box size="${d435_cam_depth} ${d435_cam_width} ${d435_cam_height}" />
           </geometry>
-          <material name="aluminum"/>
+          <material name="aluminum" />
         </xacro:unless>
       </visual>
       <collision>
-        <origin xyz="0 ${-d435_cam_depth_py} 0" rpy="0 0 0"/>
+        <origin xyz="0 ${-d435_cam_depth_py} 0" rpy="0 0 0" />
         <geometry>
-          <box size="${d435_cam_depth} ${d435_cam_width} ${d435_cam_height}"/>
+          <box size="${d435_cam_depth} ${d435_cam_width} ${d435_cam_height}" />
         </geometry>
       </collision>
@@ -78,13 +81,14 @@
       </inertial>
     </link>
-    <!-- Use the nominal extrinsics between camera frames if the calibrated extrinsics aren't being published. e.g. running the device in simulation  -->
+    <!-- Use the nominal extrinsics between camera frames if the calibrated extrinsics aren't being
+    published. e.g. running the device in simulation  -->
     <xacro:if value="${use_nominal_extrinsics}">
       <!-- camera depth joints and links -->
       <joint name="${name}_depth_joint" type="fixed">
-        <origin xyz="0 0 0" rpy="0 0 0"/>
-        <parent link="${name}_link"/>
+        <origin xyz="0 0 0" rpy="0 0 0" />
+        <parent link="${name}_link" />
         <child link="${name}_depth_frame" />
       </joint>
-      <link name="${name}_depth_frame"/>
+      <link name="${name}_depth_frame" />
       <joint name="${name}_depth_optical_joint" type="fixed">
         <origin xyz="0 0 0" rpy="${-M_PI/2} 0 ${-M_PI/2}" />
@@ -92,5 +96,5 @@
         <child link="${name}_depth_optical_frame" />
       </joint>
-      <link name="${name}_depth_optical_frame"/>
+      <link name="${name}_depth_optical_frame" />
       <!-- camera left IR joints and links -->
       <joint name="${name}_infra1_joint" type="fixed">
@@ -99,5 +103,5 @@
         <child link="${name}_infra1_frame" />
       </joint>
-      <link name="${name}_infra1_frame"/>
+      <link name="${name}_infra1_frame" />
       <joint name="${name}_infra1_optical_joint" type="fixed">
         <origin xyz="0 0 0" rpy="${-M_PI/2} 0 ${-M_PI/2}" />
@@ -105,5 +109,5 @@
         <child link="${name}_infra1_optical_frame" />
       </joint>
-      <link name="${name}_infra1_optical_frame"/>
+      <link name="${name}_infra1_optical_frame" />
       <!-- camera right IR joints and links -->
       <joint name="${name}_infra2_joint" type="fixed">
@@ -112,5 +116,5 @@
         <child link="${name}_infra2_frame" />
       </joint>
-      <link name="${name}_infra2_frame"/>
+      <link name="${name}_infra2_frame" />
       <joint name="${name}_infra2_optical_joint" type="fixed">
         <origin xyz="0 0 0" rpy="${-M_PI/2} 0 ${-M_PI/2}" />
@@ -118,5 +122,5 @@
         <child link="${name}_infra2_optical_frame" />
       </joint>
-      <link name="${name}_infra2_optical_frame"/>
+      <link name="${name}_infra2_optical_frame" />
       <!-- camera color joints and links -->
       <joint name="${name}_color_joint" type="fixed">
@@ -125,5 +129,5 @@
         <child link="${name}_color_frame" />
       </joint>
-      <link name="${name}_color_frame"/>
+      <link name="${name}_color_frame" />
       <joint name="${name}_color_optical_joint" type="fixed">
         <origin xyz="0 0 0" rpy="${-M_PI/2} 0 ${-M_PI/2}" />
@@ -131,13 +135,20 @@
         <child link="${name}_color_optical_frame" />
       </joint>
-      <link name="${name}_color_optical_frame"/>
+      <link name="${name}_color_optical_frame" />
     </xacro:if>
     <xacro:if value="${add_plug}">
       <xacro:usb_plug parent="${name}_link" name="${name}_usb_plug">
-        <origin xyz="${d435_cam_mount_from_center_offset - 0.02095} ${-d435_cam_depth_py - 0.0353} 0" rpy="0 0 0"/>
+        <origin
+          xyz="${d435_cam_mount_from_center_offset - 0.02095} ${-d435_cam_depth_py - 0.0353} 0"
+          rpy="0 0 0" />
       </xacro:usb_plug>
     </xacro:if>
     <!-- Realsense Gazebo Plugin -->
-    <xacro:gazebo_d435 camera_name="${name}" reference_link="${name}_link" topics_ns="${topics_ns}" depth_optical_frame="${name}_depth_optical_frame" color_optical_frame="${name}_color_optical_frame" infrared1_optical_frame="${name}_left_ir_optical_frame" infrared2_optical_frame="${name}_right_ir_optical_frame" publish_pointcloud="${publish_pointcloud}"/>
+    <xacro:gazebo_d435 camera_name="${name}" reference_link="${name}_link" topics_ns="${topics_ns}"
+      depth_optical_frame="${name}_depth_optical_frame"
+      color_optical_frame="${name}_color_optical_frame"
+      infrared1_optical_frame="${name}_left_ir_optical_frame"
+      infrared2_optical_frame="${name}_right_ir_optical_frame"
+      publish_pointcloud="${publish_pointcloud}" />
   </xacro:macro>
 </robot>

File: src/realsense-ros-gazebo/realsense-ros/realsense2_description/urdf/test_d435_camera.urdf.xacro (robot description, xacro)
@@ -1,5 +1,5 @@
 <?xml version="1.0"?>
 <robot name="realsense2_camera" xmlns:xacro="http://ros.org/wiki/xacro">
-  <xacro:arg name="use_nominal_extrinsics" default="false"/>
+  <xacro:arg name="use_nominal_extrinsics" default="false" />
   <xacro:arg name="add_plug" default="false" />
   <xacro:arg name="use_mesh" default="true" />
@@ -9,6 +9,8 @@
   <xacro:include filename="$(find realsense2_description)/urdf/_d435.urdf.xacro" />
   <link name="base_link" />
-  <xacro:sensor_d435 parent="base_link" use_nominal_extrinsics="$(arg use_nominal_extrinsics)" add_plug="$(arg add_plug)" use_mesh="$(arg use_mesh)" name="$(arg name)" topics_ns="$(arg topics_ns)" publish_pointcloud="$(arg publish_pointcloud)">
-    <origin xyz="0 0 0" rpy="0 0 0"/>
+  <xacro:sensor_d435 parent="base_link" use_nominal_extrinsics="$(arg use_nominal_extrinsics)"
+    add_plug="$(arg add_plug)" use_mesh="$(arg use_mesh)" name="$(arg name)"
+    topics_ns="$(arg topics_ns)" publish_pointcloud="$(arg publish_pointcloud)">
+    <origin xyz="0 0 0" rpy="0 0 0" />
   </xacro:sensor_d435>
 </robot>

File: src/umbot/urdf/mybot.xacro (robot description, xacro)
@@ -169,22 +169,35 @@
   <!--   <origin rpy="0 0 0 " xyz="0.10 0 0.025" /> -->
   <!-- </xacro:realsense_d435> -->
-  <xacro:sensor_d455 name="camera" parent="base_link">
+  <!-- <xacro:sensor_d455 name="camera" parent="base_link"> -->
+  <!--   <origin xyz="0.1 0 0.025" rpy="0 0 0" /> -->
+  <!-- </xacro:sensor_d455> -->
+  <xacro:arg name="use_nominal_extrinsics" default="false" />
+  <xacro:arg name="add_plug" default="false" />
+  <xacro:arg name="use_mesh" default="true" />
+  <xacro:arg name="name" default="camera" />
+  <xacro:arg name="topics_ns" default="camera" />
+  <xacro:arg name="publish_pointcloud" default="true" />
+  <xacro:include filename="$(find realsense2_description)/urdf/_d435.urdf.xacro" />
+  <xacro:sensor_d435 parent="base_link" use_nominal_extrinsics="$(arg use_nominal_extrinsics)"
+    add_plug="$(arg add_plug)" use_mesh="$(arg use_mesh)" name="$(arg name)"
+    topics_ns="$(arg topics_ns)" publish_pointcloud="$(arg publish_pointcloud)">
     <origin xyz="0.1 0 0.025" rpy="0 0 0" />
-  </xacro:sensor_d455>
+  </xacro:sensor_d435>
   <!-- lidar sensor -->
-  <link name="lidar">
-    <visual>
-      <geometry>
-        <box size="0.05 0.05 0.05" />
-      </geometry>
-      <material name="white">
-        <color rgba="1 1 1 1 " />
-      </material>
-    </visual>
-  </link>
-  <joint name="lidar_joint" type="fixed">
-    <parent link="base_link" />
-    <child link="lidar" />
-    <origin xyz="0.10 0 0.065" />
-  </joint>
+  <!-- <link name="lidar"> -->
+  <!--   <visual> -->
+  <!--     <geometry> -->
+  <!--       <box size="0.05 0.05 0.05" /> -->
+  <!--     </geometry> -->
+  <!--     <material name="white"> -->
+  <!--       <color rgba="1 1 1 1 " /> -->
+  <!--     </material> -->
+  <!--   </visual> -->
+  <!-- </link> -->
+  <!---->
+  <!-- <joint name="lidar_joint" type="fixed"> -->
+  <!--   <parent link="base_link" /> -->
+  <!--   <child link="lidar" /> -->
+  <!--   <origin xyz="0.10 0 0.065" /> -->
+  <!-- </joint> -->
 </robot>
