Commit message: bugfix(laser tf work)

File: src/umbot/urdf/mybot.gazebo.xacro (robot description, xacro)
@@ -1,4 +1,59 @@
 <?xml version="1.0"?>
 <robot name="mybot" xmlns:xacro="http://ros.org/wiki/xacro">
+  <xacro:macro name="null_inertial">
+    <inertial>
+      <mass value="0.1"/>
+      <inertia ixx="0.01" ixy="0" ixz="0"
+        iyy="0.01" iyz="0"
+        izz="0.01"/>
+    </inertial>
+  </xacro:macro>
+  <xacro:property name="M_PI" value="3.14159"/>
+  <xacro:property name="laser_min_range" value="0.1"/>
+  <xacro:property name="laser_max_range" value="200.0"/>
+  <xacro:property name="ros_topic" value="scan"/>
+  <xacro:property name="samples" value="24000"/>
+  <xacro:property name="downsample" value="1"/>
+  <gazebo reference="laser_livox">
+    <sensor type="ray" name="laser_livox">
+      <pose>0 0 0 0 0 0</pose>
+      <visualize>true</visualize>
+      <update_rate>10</update_rate>
+      <!-- This ray plgin is only for visualization. -->
+      <plugin name="gazebo_ros_laser_controller" filename="liblivox_laser_simulation.so">
+        <ray>
+          <scan>
+            <horizontal>
+              <samples>100</samples>
+              <resolution>1</resolution>
+              <min_angle>${0}</min_angle>
+              <max_angle>${2*M_PI}</max_angle>
+            </horizontal>
+            <vertical>
+              <samples>360</samples>
+              <resolution>1</resolution>
+              <min_angle>${-7.22/180*M_PI}</min_angle>
+              <max_angle>${55.22/180*M_PI}</max_angle>
+            </vertical>
+          </scan>
+          <range>
+            <min>${laser_min_range}</min>
+            <max>${laser_max_range}</max>
+            <resolution>0.002</resolution>
+          </range>
+          <noise>
+            <type>gaussian</type>
+            <mean>0.0</mean>
+            <stddev>0.01</stddev>
+          </noise>
+        </ray>
+        <visualize>true</visualize>
+        <samples>24000</samples>
+        <downsample>1</downsample>
+        <csv_file_name>package://livox_laser_simulation/scan_mode/mid360.csv</csv_file_name>
+        <ros_topic>scan</ros_topic>
+      </plugin>
+    </sensor>
+  </gazebo>
   <gazebo>
     <plugin name="skid_steer_drive_controller" filename="libgazebo_ros_skid_steer_drive.so">

File: src/umbot/urdf/mybot.xacro (robot description, xacro)
@@ -1,11 +1,12 @@
 <?xml version="1.0"?>
-<robot name="mybot" xmlns:xacro="http://ros.org/wiki/xacro">
+<robot name="mybot" xmlns:xacro="http://ros.org/wiki/xacro" >
   <xacro:include filename="$(find realsense2_description)/urdf/_d455.urdf.xacro" />
   <xacro:include filename="$(find umbot)/urdf/mybot.gazebo.xacro" />
   <link name="base_footprint" />
-  <joint name="base_joint" type="fixed">
+  <joint name="base_link_footprint" type="fixed">
+    <axis xyz="0 0 0" />
     <parent link="base_footprint" />
     <child link="base_link" />
-    <origin rpy="0 0 0" xyz="0 0 0" />
+    <origin rpy="0 0 0" xyz=" 0 0 0" />
   </joint>
   <link name="base_link">
@@ -149,27 +150,4 @@
     <origin xyz="0.08 0 0.025" />
   </joint>
-  <!-- camera sensor -->
-  <!-- <link name="camera"> -->
-  <!--   <visual> -->
-  <!--     <geometry> -->
-  <!--       <box size="0.02 0.08 0.03" /> -->
-  <!--     </geometry> -->
-  <!--     <material name="white"> -->
-  <!--       <color rgba="1 1 1 1 " /> -->
-  <!--     </material> -->
-  <!--   </visual> -->
-  <!-- </link> -->
-  <!---->
-  <!-- <joint name="camera_joint" type="fixed"> -->
-  <!--   <parent link="base_link" /> -->
-  <!--   <child link="camera" /> -->
-  <!--   <origin xyz="0.10 0 0.025" /> -->
-  <!-- </joint> -->
-  <!-- <xacro:realsense_d435 sensor_name="d435" parent_link="base_link" rate="10"> -->
-  <!--   <origin rpy="0 0 0 " xyz="0.10 0 0.025" /> -->
-  <!-- </xacro:realsense_d435> -->
-  <!-- <xacro:sensor_d455 name="camera" parent="base_link"> -->
-  <!--   <origin xyz="0.1 0 0.025" rpy="0 0 0" /> -->
-  <!-- </xacro:sensor_d455> -->
   <xacro:arg name="use_nominal_extrinsics" default="false" />
   <xacro:arg name="add_plug" default="false" />
@@ -182,22 +160,26 @@
     add_plug="$(arg add_plug)" use_mesh="$(arg use_mesh)" name="$(arg name)"
     topics_ns="$(arg topics_ns)" publish_pointcloud="$(arg publish_pointcloud)">
-    <origin xyz="0.1 0 0.025" rpy="0 0 0" />
-  </xacro:sensor_d435>
-  <!-- lidar sensor -->
-  <!-- <link name="lidar"> -->
-  <!--   <visual> -->
-  <!--     <geometry> -->
-  <!--       <box size="0.05 0.05 0.05" /> -->
-  <!--     </geometry> -->
-  <!--     <material name="white"> -->
-  <!--       <color rgba="1 1 1 1 " /> -->
-  <!--     </material> -->
-  <!--   </visual> -->
-  <!-- </link> -->
-  <!---->
-  <!-- <joint name="lidar_joint" type="fixed"> -->
-  <!--   <parent link="base_link" /> -->
-  <!--   <child link="lidar" /> -->
-  <!--   <origin xyz="0.10 0 0.065" /> -->
-  <!-- </joint> -->
-</robot>
+  <origin xyz="0.1 0 0.025" rpy="0 0 0" />
+</xacro:sensor_d435>
+<link name="laser_livox">
+  <xacro:null_inertial/>
+  <visual>
+    <origin xyz="0.00 0 0.0" rpy="0 0 0"/>
+    <geometry>
+      <mesh filename="package://livox_laser_simulation/meshes/livox_mid40.dae">
+      </mesh>
+    </geometry>
+  </visual>
+  <collision>
+    <origin xyz="0 0 0" rpy="0 0 0" />
+    <geometry>
+      <mesh filename="package://livox_laser_simulation/meshes/livox_mid40.dae"/>
+    </geometry>
+  </collision>
+</link>
+<joint name="$livox_to_base_joint" type="fixed">
+  <parent link="base_link"/>
+  <child link="laser_livox"/>
+  <origin rpy="0 0 0" xyz="0.0 0.0 0.05"/>
+</joint>
+  </robot>
